File: PCB/PCB.kicad_pcb (KiCad board)
At the start: 2 copper layers, 95 x 71.5 mm, 41 parts, among them J1 Conn_01x02, J2 Conn_01x02, J3 Conn_01x03, U1 Seeed Studio XIAO nRF52840, U2 Seeed Studio XIAO nRF52840

Commit message: first
Routing:
- net /Row3: track 136.3 -> 139.9 mm
- net /Row2: track 141.0 -> 141.7 mm
Other:
- outline, holes or cut-outs redrawn
Changed lines of the file:
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@@
 		(layer "Edge.Cuts")
 	)
+	(gr_circle
+		(center 99 42.5)
+		(end 101 42.5)
+		(stroke
+			(width 0.05)
+			(type default)
+		)
+		(fill none)
+		(layer "Edge.Cuts")
+	)
 	(gr_arc
 		(start 116 23.5)
@@
 		(layer "Edge.Cuts")
 	)
+	(gr_circle
+		(center 45 51)
+		(end 47 51)
+		(stroke
+			(width 0.05)
+			(type default)
+		)
+		(fill none)
+		(layer "Edge.Cuts")
+	)
 	(gr_line
 		(start 116 23.5)
@@
 		(layer "Edge.Cuts")
 	)
+	(gr_circle
+		(center 99 76.5)
+		(end 101 76.5)
+		(stroke
+			(width 0.05)
+			(type default)
+		)
+		(fill none)
+		(layer "Edge.Cuts")
+	)
+	(gr_circle
+		(center 45 76.5)
+		(end 47 76.5)
+		(stroke
+			(width 0.05)
+			(type default)
+		)
+		(fill none)
+		(layer "Edge.Cuts")
+	)
 	(gr_line
 		(start 116 95)
@@
 	)
 	(segment
+		(start 47.1 48.844491)
+		(end 47.1 34.562974)
+		(width 0.2)
+		(layer "F.Cu")
+		(net 6)
+	)
+	(segment
 		(start 41.1 31.325735)
 		(end 40.574265 30.8)
@@
 	)
 	(segment
-		(start 28.672015 31.5)
-		(end 27.5 32.672015)
+		(start 47.1 70.5)
+		(end 47.1 53.315686)
 		(width 0.2)
 		(layer "F.Cu")
@@
 	)
 	(segment
-		(start 47.1 70.5)
-		(end 47.1 34.562974)
+		(start 48.001681 52.414005)
+		(end 48.001681 49.746171)
+		(width 0.2)
+		(layer "F.Cu")
+		(net 6)
+	)
+	(segment
+		(start 28.672015 31.5)
+		(end 27.5 32.672015)
 		(width 0.2)
 		(layer "F.Cu")
@@
 	)
 	(segment
-		(start 47.1 34.562974)
-		(end 46.442272 33.905246)
+		(start 48.001681 49.746171)
+		(end 47.767366 49.511857)
+		(width 0.2)
+		(layer "F.Cu")
+		(net 6)
+	)
+	(segment
+		(start 47.1 53.315686)
+		(end 48.001681 52.414005)
 		(width 0.2)
 		(layer "F.Cu")
@@
 	)
 	(segment
+		(start 47.1 34.562974)
+		(end 46.442272 33.905246)
+		(width 0.2)
+		(layer "F.Cu")
+		(net 6)
+	)
+	(segment
 		(start 38.9 31.151471)
 		(end 38.9 31.5)
@@
 	)
 	(segment
+		(start 47.767366 49.511857)
+		(end 47.1 48.844491)
+		(width 0.2)
+		(layer "F.Cu")
+		(net 6)
+	)
+	(segment
 		(start 38.9 31.5)
 		(end 28.672015 31.5)
@@
 	)
 	(segment
-		(start 45.725 80.25)
-		(end 45.725 77.576671)
+		(start 49.775 84.3)
+		(end 59.325 84.3)
 		(width 0.2)
 		(layer "B.Cu")
@@
 	)
 	(segment
-		(start 51.051671 72.25)
-		(end 52.35 72.25)
+		(start 48.2741 77.7009)
+		(end 48.997429 77.7009)
 		(width 0.2)
 		(layer "B.Cu")
@@
 	)
 	(segment
-		(start 49.775 84.3)
-		(end 59.325 84.3)
+		(start 48.997429 77.7009)
+		(end 52.35 74.348329)
 		(width 0.2)
 		(layer "B.Cu")
@@
 	)
 	(segment
-		(start 45.725 77.576671)
-		(end 51.051671 72.25)
+		(start 45.725 80.25)
+		(end 48.2741 77.7009)
 		(width 0.2)
 		(layer "B.Cu")
@@
 		(net 9)
 	)
+	(segment
+		(start 52.35 74.348329)
+		(end 52.35 72.25)
+		(width 0.2)
+		(layer "B.Cu")
+		(net 9)
+	)
 	(via
 		(at 79.924998 37.75)
@@
 	)
 	(segment
-		(start 45.5 83.5)
-		(end 45.875 83.125)
+		(start 46.5 48.810176)
+		(end 47.601681 49.911857)
 		(width 0.2)
 		(layer "F.Cu")
@@
 	)
 	(segment
-		(start 46.5 61.616295)
-		(end 46.5 36.5)
+		(start 28.447852 36.159867)
+		(end 27.5 35.212015)
 		(width 0.2)
 		(layer "F.Cu")
@@
 	)
 	(segment
-		(start 28.447852 36.159867)
-		(end 27.5 35.212015)
+		(start 45.875 80.758705)
+		(end 45.875 83.125)
 		(width 0.2)
 		(layer "F.Cu")
@@
 	)
 	(segment
-		(start 45.875 83.125)
-		(end 45.875 62.241295)
+		(start 49.7009 76.002571)
+		(end 49.7009 76.997429)
 		(width 0.2)
 		(layer "F.Cu")
@@
 	)
 	(segment
-		(start 45.875 62.241295)
-		(end 46.5 61.616295)
+		(start 48.298329 78.4)
+		(end 48.233705 78.4)
+		(width 0.2)
+		(layer "F.Cu")
+		(net 36)
+	)
+	(segment
+		(start 45.875 83.125)
+		(end 45.5 83.5)
 		(width 0.2)
 		(layer "F.Cu")
@@
 		(width 0.2)
 		(layer "F.Cu")
+		(net 36)
+	)
+	(segment
+		(start 49.7009 76.997429)
+		(end 48.298329 78.4)
+		(width 0.2)
+		(layer "F.Cu")
+		(net 36)
+	)
+	(segment
+		(start 47.601681 52.248319)
+		(end 46.5 53.35)
+		(width 0.2)
+		(layer "F.Cu")
+		(net 36)
+	)
+	(segment
+		(start 46.5 36.5)
+		(end 46.5 48.810176)
+		(width 0.2)
+		(layer "F.Cu")
+		(net 36)
+	)
+	(segment
+		(start 48.233705 78.4)
+		(end 45.875 80.758705)
+		(width 0.2)
+		(layer "F.Cu")
+		(net 36)
+	)
+	(segment
+		(start 46.5 72.801671)
+		(end 49.7009 76.002571)
+		(width 0.2)
+		(layer "F.Cu")
+		(net 36)
+	)
+	(segment
+		(start 47.601681 49.911857)
+		(end 47.601681 52.248319)
+		(width 0.2)
+		(layer "F.Cu")
+		(net 36)
+	)
+	(segment
+		(start 46.5 53.35)
+		(end 46.5 72.801671)
+		(width 0.2)
+		(layer "F.Cu")

Commit message: pcb v0.1
Parts:
- added D7: D_Schottky, Diode_SMD:D_SMA, B.Cu at (53.6, 25.6)
Connections:
- J3 pad 1: +5V -> Net-(D7-K)
Routing:
- net +5V: track 120.3 -> 25.4 mm
- net Net-(D7-K): track 0.00 -> 91.6 mm
- net Net-(D3-A): track 24.5 -> 32.1 mm
- net /Col3: track 218.0 -> 220.6 mm
- net /Bat-: vias 1 -> 0
- net /Bat+: vias 1 -> 0
Other:
- outline, holes or cut-outs redrawn
- board text added: "Board: PickPocket Version: 0.1 Developer: Parks Date: 02/19/25"
- board text removed: "Board: PickPocket Version: 0.1 Developer: Parks Date: 02/12/25"
